Commit message: Add gazebo

File: motoman_sda10f_support/urdf/arm_macro.xacro (robot description, xacro)
@@ -18,4 +18,9 @@
         </geometry>
       </collision>
+      <inertial>
+            <mass value="0.5" />
+            <origin xyz="0 0 0" rpy="0 0 0" />
+            <inertia ixx="0.004" ixy="0.001" ixz="0" iyy="0.006" iyz="0" izz="0.007" />
+        </inertial>
     </link>
     <link name="${prefix}link_2_l">
@@ -33,4 +38,9 @@
         </geometry>
       </collision>
+      <inertial>
+            <mass value="0.5" />
+            <origin xyz="0 0 0" rpy="0 0 0" />
+            <inertia ixx="0.004" ixy="0.001" ixz="0" iyy="0.006" iyz="0" izz="0.007" />
+        </inertial>
     </link>
     <link name="${prefix}link_3_e">
@@ -48,4 +58,9 @@
         </geometry>
       </collision>
+      <inertial>
+            <mass value="0.5" />
+            <origin xyz="0 0 0" rpy="0 0 0" />
+            <inertia ixx="0.004" ixy="0.001" ixz="0" iyy="0.006" iyz="0" izz="0.007" />
+        </inertial>
     </link>
     <link name="${prefix}link_4_u">
@@ -63,4 +78,9 @@
         </geometry>
       </collision>
+      <inertial>
+            <mass value="0.5" />
+            <origin xyz="0 0 0" rpy="0 0 0" />
+            <inertia ixx="0.004" ixy="0.001" ixz="0" iyy="0.006" iyz="0" izz="0.007" />
+        </inertial>
     </link>
     <link name="${prefix}link_5_r">
@@ -78,4 +98,9 @@
         </geometry>
       </collision>
+      <inertial>
+            <mass value="0.5" />
+            <origin xyz="0 0 0" rpy="0 0 0" />
+            <inertia ixx="0.004" ixy="0.001" ixz="0" iyy="0.006" iyz="0" izz="0.007" />
+        </inertial>
     </link>
     <link name="${prefix}link_6_b">
@@ -93,4 +118,9 @@
         </geometry>
       </collision>
+        <inertial>
+            <mass value="0.5" />
+            <origin xyz="0 0 0" rpy="0 0 0" />
+            <inertia ixx="0.004" ixy="0.001" ixz="0" iyy="0.006" iyz="0" izz="0.007" />
+        </inertial>
     </link>
     <link name="${prefix}link_7_t">
@@ -106,4 +136,9 @@
         </geometry>
       </collision>
+      <inertial>
+            <mass value="0.5" />
+            <origin xyz="0 0 0" rpy="0 0 0" />
+            <inertia ixx="0.004" ixy="0.001" ixz="0" iyy="0.006" iyz="0" izz="0.007" />
+        </inertial>
     </link>
     <link name="${prefix}link_tool0" />

File: motoman_sda10f_support/urdf/common_torso_macro.xacro (robot description, xacro)
@@ -17,4 +17,9 @@
         </geometry>
       </collision>
+      <inertial>
+            <mass value="5" />
+            <origin xyz="0 0 0" rpy="0 0 0" />
+            <inertia ixx="0.004" ixy="0.001" ixz="0" iyy="0.006" iyz="0" izz="0.007" />
+        </inertial>
     </link>
     <link name="${prefix}link_b1">
@@ -34,4 +39,9 @@
         </geometry>
       </collision>
+      <inertial>
+            <mass value="5" />
+            <origin xyz="0 0 0" rpy="0 0 0" />
+            <inertia ixx="0.004" ixy="0.001" ixz="0" iyy="0.006" iyz="0" izz="0.007" />
+        </inertial>
     </link>
     <link name="${prefix}link_b2"/>

Commit message: Add move group to test.launch

File: motoman_sda10f_support/urdf/arm_macro.xacro (robot description, xacro)
@@ -19,8 +19,13 @@
       </collision>
       <inertial>
-            <mass value="0.5" />
-            <origin xyz="0 0 0" rpy="0 0 0" />
-            <inertia ixx="0.004" ixy="0.001" ixz="0" iyy="0.006" iyz="0" izz="0.007" />
-        </inertial>
+        <mass value="0.01" />
+        <inertia
+          ixx="0.00950655468"
+          ixy="0"
+          ixz="0"
+          iyy="0.0054345236"
+          iyz="0"
+          izz="0.01148428921" />
+      </inertial>
     </link>
     <link name="${prefix}link_2_l">
@@ -39,7 +44,12 @@
       </collision>
       <inertial>
-            <mass value="0.5" />
-            <origin xyz="0 0 0" rpy="0 0 0" />
-            <inertia ixx="0.004" ixy="0.001" ixz="0" iyy="0.006" iyz="0" izz="0.007" />
+        <mass value="0.01" />
+        <inertia
+          ixx="0.00950655468"
+          ixy="0"
+          ixz="0"
+          iyy="0.0054345236"
+          iyz="0"
+          izz="0.01148428921" />
         </inertial>
     </link>
@@ -59,7 +69,12 @@
       </collision>
       <inertial>
-            <mass value="0.5" />
-            <origin xyz="0 0 0" rpy="0 0 0" />
-            <inertia ixx="0.004" ixy="0.001" ixz="0" iyy="0.006" iyz="0" izz="0.007" />
+        <mass value="0.01" />
+        <inertia
+          ixx="0.00950655468"
+          ixy="0"
+          ixz="0"
+          iyy="0.0054345236"
+          iyz="0"
+          izz="0.01148428921" />
         </inertial>
     </link>
@@ -79,7 +94,12 @@
       </collision>
       <inertial>
-            <mass value="0.5" />
-            <origin xyz="0 0 0" rpy="0 0 0" />
-            <inertia ixx="0.004" ixy="0.001" ixz="0" iyy="0.006" iyz="0" izz="0.007" />
+        <mass value="0.01" />
+        <inertia
+          ixx="0.00950655468"
+          ixy="0"
+          ixz="0"
+          iyy="0.0054345236"
+          iyz="0"
+          izz="0.01148428921" />
         </inertial>
     </link>
@@ -99,7 +119,12 @@
       </collision>
       <inertial>
-            <mass value="0.5" />
-            <origin xyz="0 0 0" rpy="0 0 0" />
-            <inertia ixx="0.004" ixy="0.001" ixz="0" iyy="0.006" iyz="0" izz="0.007" />
+        <mass value="0.01" />
+        <inertia
+          ixx="0.00950655468"
+          ixy="0"
+          ixz="0"
+          iyy="0.0054345236"
+          iyz="0"
+          izz="0.01148428921" />
         </inertial>
     </link>
@@ -119,7 +144,12 @@
       </collision>
         <inertial>
-            <mass value="0.5" />
-            <origin xyz="0 0 0" rpy="0 0 0" />
-            <inertia ixx="0.004" ixy="0.001" ixz="0" iyy="0.006" iyz="0" izz="0.007" />
+        <mass value="0.01" />
+        <inertia
+          ixx="0.00950655468"
+          ixy="0"
+          ixz="0"
+          iyy="0.0054345236"
+          iyz="0"
+          izz="0.01148428921" />
         </inertial>
     </link>
@@ -137,7 +167,12 @@
       </collision>
       <inertial>
-            <mass value="0.5" />
-            <origin xyz="0 0 0" rpy="0 0 0" />
-            <inertia ixx="0.004" ixy="0.001" ixz="0" iyy="0.006" iyz="0" izz="0.007" />
+        <mass value="0.01" />
+        <inertia
+          ixx="0.00950655468"
+          ixy="0"
+          ixz="0"
+          iyy="0.0054345236"
+          iyz="0"
+          izz="0.01148428921" />
         </inertial>
     </link>
